File: jlcmotor/jlcmotor.kicad_pcb (KiCad board)
At the start: 2 copper layers, 96.5 x 66 mm, 19 parts, among them J1 ScrewTerminal, U1 PinHeader8, U2 PinHeader8

Commit message: bulk capacitor
Parts:
- added C1: ~, Capacitor_SMD:C_1206_3216Metric, F.Cu at (96.5, 35.6)
Routing:
- net /VMOT: track 72.4 -> 78.0 mm
- net /GND: track 238.1 -> 241.1 mm, vias 0 -> 1
Changed lines of the file:
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@@
 	(net 31 "Net-(U2-Pin_4)")
 	(net 32 "/3V3")
+	(footprint "Capacitor_SMD:C_1206_3216Metric"
+		(layer "F.Cu")
+		(at 96.52 35.56 -90)
+		(descr "Capacitor SMD 1206 (3216 Metric), square (rectangular) end terminal, IPC-7351 nominal, (Body size source: IPC-SM-782 page 76, https://www.pcb-3d.com/wordpress/wp-content/uploads/ipc-sm-782a_amendment_1_and_2.pdf), generated with kicad-footprint-generator")
+		(tags "capacitor")
+		(property "Reference" "C1"
+			(at 0 -1.85 90)
+			(layer "F.SilkS")
+			(effects
+				(font
+					(size 1 1)
+					(thickness 0.15)
+				)
+			)
+		)
+		(property "Value" "~"
+			(at 0 1.85 90)
+			(layer "F.Fab")
+			(effects
+				(font
+					(size 1 1)
+					(thickness 0.15)
+				)
+			)
+		)
+		(property "Datasheet" ""
+			(at 0 0 90)
+			(layer "F.Fab")
+			(hide yes)
+			(effects
+				(font
+					(size 1.27 1.27)
+					(thickness 0.15)
+				)
+			)
+		)
+		(property "Description" ""
+			(at 0 0 90)
+			(layer "F.Fab")
+			(hide yes)
+			(effects
+				(font
+					(size 1.27 1.27)
+					(thickness 0.15)
+				)
+			)
+		)
+		(property "lcsc" "C76659"
+			(at 0 0 270)
+			(unlocked yes)
+			(layer "F.Fab")
+			(hide yes)
+			(effects
+				(font
+					(size 1 1)
+					(thickness 0.15)
+				)
+			)
+		)
+		(property ki_fp_filters "C_*")
+		(sheetname "/")
+		(sheetfile "jlcmotor.kicad_sch")
+		(attr smd)
+		(fp_line
+			(start -0.711252 0.91)
+			(end 0.711252 0.91)
+			(stroke
+				(width 0.12)
+				(type solid)
+			)
+			(layer "F.SilkS")
+		)
+		(fp_line
+			(start -0.711252 -0.91)
+			(end 0.711252 -0.91)
+			(stroke
+				(width 0.12)
+				(type solid)
+			)
+			(layer "F.SilkS")
+		)
+		(fp_rect
+			(start -2.3 -1.15)
+			(end 2.3 1.15)
+			(stroke
+				(width 0.05)
+				(type solid)
+			)
+			(fill no)
+			(layer "F.CrtYd")
+		)
+		(fp_rect
+			(start -1.6 -0.8)
+			(end 1.6 0.8)
+			(stroke
+				(width 0.1)
+				(type solid)
+			)
+			(fill no)
+			(layer "F.Fab")
+		)
+		(fp_text user "${REFERENCE}"
+			(at 0 0 90)
+			(layer "F.Fab")
+			(effects
+				(font
+					(size 0.8 0.8)
+					(thickness 0.12)
+				)
+			)
+		)
+		(pad "1" smd roundrect
+			(at -1.475 0 270)
+			(size 1.15 1.8)
+			(layers "F.Cu" "F.Mask" "F.Paste")
+			(roundrect_rratio 0.217391)
+			(net 3 "/VMOT")
+			(pintype "passive")
+		)
+		(pad "2" smd roundrect
+			(at 1.475 0 270)
+			(size 1.15 1.8)
+			(layers "F.Cu" "F.Mask" "F.Paste")
+			(roundrect_rratio 0.217391)
+			(net 24 "/GND")
+			(pintype "passive")
+		)
+		(embedded_fonts no)
+		(model "${KICAD9_3DMODEL_DIR}/Capacitor_SMD.3dshapes/C_1206_3216Metric.step"
+			(offset
+				(xyz 0 0 0)
+			)
+			(scale
+				(xyz 1 1 1)
+			)
+			(rotate
+				(xyz 0 0 0)
+			)
+		)
+	)
 	(footprint "Connector_PinSocket_2.54mm:PinSocket_1x04_P2.54mm_Vertical"
 		(layer "F.Cu")
@@
 	)
 	(segment
+		(start 96.52 34.085)
+		(end 92.915 34.085)
+		(width 0.2)
+		(layer "F.Cu")
+		(net 3)
+	)
+	(segment
 		(start 88.9 71.12)
 		(end 78.74 81.28)
@@
 	)
 	(segment
+		(start 92.915 34.085)
+		(end 91.44 35.56)
+		(width 0.2)
+		(layer "F.Cu")
+		(net 3)
+	)
+	(segment
 		(start 91.44 48.26)
 		(end 96.52 53.34)
@@
 	)
 	(segment
+		(start 95.045 37.035)
+		(end 93.98 38.1)
+		(width 0.2)
+		(layer "F.Cu")
+		(net 24)
+	)
+	(segment
 		(start 30.48 38.1)
 		(end 38.1 30.48)
@@
 	)
 	(segment
+		(start 96.52 37.035)
+		(end 95.045 37.035)
+		(width 0.2)
+		(layer "F.Cu")
+		(net 24)
+	)
+	(segment
 		(start 33.02 74.168)
 		(end 33.02 71.628)
@@
 		(net 24)
 	)
+	(via
+		(at 93.98 38.1)
+		(size 0.6)
+		(drill 0.3)
+		(layers "F.Cu" "B.Cu")
+		(net 24)
+	)

Commit message: limit sw
Parts:
- added C2: ~, Capacitor_SMD:C_0603_1608Metric, F.Cu at (78.7, 81.3)
- added C3: ~, Capacitor_SMD:C_0603_1608Metric, F.Cu at (88.9, 81.3)
- added R2: ~, Resistor_SMD:R_0603_1608Metric, F.Cu at (78.7, 76.2)
- added R3: ~, Resistor_SMD:R_0603_1608Metric, F.Cu at (88.9, 76.2)
Connections:
- J2 pad 3: /<NO NET> -> unconnected-(J2-Pin_3-Pad3)
- J2 pad 4: /<NO NET> -> unconnected-(J2-Pin_4-Pad4)
- J3 pad 1: unconnected-(J3-Pin_1-Pad1) -> /GND
- J3 pad 2: unconnected-(J3-Pin_2-Pad2) -> Net-(J3-Pin_2)
- J3 pad 3: unconnected-(J3-Pin_3-Pad3) -> /GND
- J3 pad 4: unconnected-(J3-Pin_4-Pad4) -> Net-(J3-Pin_4)
- U1 pad 3: unconnected-(U1-Pin_3-Pad3) -> Net-(J3-Pin_2)
- U1 pad 7: unconnected-(U1-Pin_7-Pad7) -> Net-(J3-Pin_4)
Routing:
- net Net-(J3-Pin_2): track 0.00 -> 83.1 mm
- net Net-(J3-Pin_4): track 0.00 -> 76.3 mm
- net /GND: track 241.1 -> 290.8 mm
- net /3V3: track 51.4 -> 89.4 mm, vias 0 -> 2
- net /<NO NET>: track 5.08 -> 0.00 mm
- net (no net): track 0.00 -> 5.08 mm
- net /VMOT: track 78.0 -> 73.6 mm, vias 0 -> 1

Commit message: status led and power oring
Parts:
- added D1: ~, Diode_SMD:D_SMA, F.Cu at (27.9, 61.0)
- added J5: ~, Connector_PinSocket_2.54mm:PinSocket_1x02_P2.54mm_Vertical, F.Cu at (43.2, 58.4)
- added R4: ~, Resistor_SMD:R_0603_1608Metric, F.Cu at (35.6, 58.4)
Connections:
- U1 pad 4: unconnected-(U1-Pin_4-Pad4) -> Net-(U1-Pin_4)
- U8 pad 1: /5V -> Net-(D1-A)
- U8 pad 2: /5V -> Net-(D1-A)
Routing:
- net /3V3: track 89.4 -> 111.9 mm, vias 2 -> 3
- net /5V: track 76.1 -> 66.9 mm
- net Net-(U1-Pin_4): track 0.00 -> 7.85 mm, vias 0 -> 1
- net Net-(D1-A): track 0.00 -> 7.84 mm
- net Net-(J5-Pin_2): track 0.00 -> 4.26 mm
- net Net-(J3-Pin_2): track 83.1 -> 79.5 mm
